File: KillSwitch_pcb/KillSwitchIO.kicad_sch (KiCad schematic)
At the start: 29 parts, among them SW6 KILL1, SW7 KILL2, SW8 KILL3, SW9 KILL4, U3 MCP23017_SO

Commit message: add pullups for i2c, reannotate, update footprints
Parts:
- removed R22, R23, R24, R25, R26, R27, R28, R29, R30, R31: 120R, Resistor_THT:R_Axial_DIN0204_L3.6mm_D1.6mm_P2.54mm_Vertical, symbol Device:R_Small
- added R10, R11, R12, R13, R14, R15, R16, R17, R18, R19: 120R, Resistor_SMD:R_0805_2012Metric_Pad1.20x1.40mm_HandSolder, symbol Device:R_Small
- R20, R21: footprint Resistor_THT:R_Axial_DIN0204_L3.6mm_D1.6mm_P2.54mm_Vertical -> Resistor_SMD:R_0805_2012Metric_Pad1.20x1.40mm_HandSolder
- renumbered D23 to D10, D24 to D11, D25 to D12, D26 to D13, D15 to D2, D16 to D3, D17 to D4, D18 to D5, D19 to D6, D20 to D7, D21 to D8, D22 to D9, SW6 to SW5, SW7 to SW6, SW8 to SW7, SW9 to SW8, U3 to U2
Connections:
- net GND: now also R10.2, R11.2, R12.2, R13.2, R14.2, R15.2, R16.2, R17.2, R18.2, R19.2
- net at D6.1 (K): now also R14.1
- net at D4.1 (K): now also R12.1
- net at D12.1 (K): now also R20.1
- net at D8.1 (K): now also R16.1
- net at D9.1 (K): now also R17.1
- net at D13.1 (K): now also R21.1
- net at D7.1 (K): now also R15.1
- net at D10.1 (K): now also R18.1
- net at D2.1 (K): now also R10.1; no longer R20.1
- net at D5.1 (K): now also R13.1
- net at D3.1 (K): now also R11.1; no longer R21.1
- net at D11.1 (K): now also R19.1

Commit message: update płytki: Routing bez GND plus obrys bez zaokrągleń i przycięć
Parts:
- added C10: 100nF, Capacitor_SMD:C_0805_2012Metric_Pad1.18x1.45mm_HandSolder, symbol Device:C_Small
Connections:
- net GND: now also C10.1
- net VDD: now also C10.2
Changed lines of the file:
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@@
+	)
+	(junction
+		(at 62.23 53.34)
+		(diameter 0)
+		(color 0 0 0 0)
 	)
 	(junction
@@
 	(wire
 		(pts
-			(xy 49.53 53.34) (xy 68.58 53.34)
+			(xy 49.53 53.34) (xy 62.23 53.34)
 		)
 		(stroke
@@
 	(wire
 		(pts
+			(xy 44.45 46.99) (xy 62.23 46.99)
+		)
+		(stroke
+			(width 0)
+			(type default)
+		)
+	)
+	(wire
+		(pts
 			(xy 49.53 100.33) (xy 50.8 100.33)
 		)
@@
 	(wire
 		(pts
+			(xy 62.23 53.34) (xy 68.58 53.34)
+		)
+		(stroke
+			(width 0)
+			(type default)
+		)
+	)
+	(wire
+		(pts
 			(xy 50.8 85.09) (xy 49.53 85.09)
 		)
@@
 		(pts
 			(xy 254 74.93) (xy 254 82.55)
+		)
+		(stroke
+			(width 0)
+			(type default)
+		)
+	)
+	(wire
+		(pts
+			(xy 62.23 46.99) (xy 62.23 53.34)
 		)
 		(stroke
@@
 			)
 			(justify left bottom)
+		)
+	)
+	(label "+3.3v_ESP"
+		(at 44.45 46.99 180)
+		(effects
+			(font
+				(size 1.27 1.27)
+			)
+			(justify right bottom)
 		)
 	)
@@
 	(symbol
 		(lib_id "power:GND")
+		(at 44.45 52.07 0)
+		(unit 1)
+		(exclude_from_sim no)
+		(in_bom yes)
+		(on_board yes)
+		(dnp no)
+		(property "Reference" "#PWR026"
+			(at 44.45 58.42 0)
+			(effects
+				(font
+					(size 1.27 1.27)
+				)
+				(hide yes)
+			)
+		)
+		(property "Value" "GND"
+			(at 44.45 57.15 0)
+			(effects
+				(font
+					(size 1.27 1.27)
+				)
+			)
+		)
+		(property "Footprint" ""
+			(at 44.45 52.07 0)
+			(effects
+				(font
+					(size 1.27 1.27)
+				)
+				(hide yes)
+			)
+		)
+		(property "Datasheet" ""
+			(at 44.45 52.07 0)
+			(effects
+				(font
+					(size 1.27 1.27)
+				)
+				(hide yes)
+			)
+		)
+		(property "Description" "Power symbol creates a global label with name \"GND\" , ground"
+			(at 44.45 52.07 0)
+			(effects
+				(font
+					(size 1.27 1.27)
+				)
+				(hide yes)
+			)
+		)
+		(pin "1"
+		)
+		(instances
+			(project "KillSwitch"
+				(path "/722d8df3-08e9-470c-940d-01bb552f6a6b/dd4eb25e-e036-4865-9a65-d34df93aca5c"
+					(reference "#PWR026")
+					(unit 1)
+				)
+			)
+		)
+	)
+	(symbol
+		(lib_id "power:GND")
 		(at 148.59 100.33 0)
 		(mirror y)
@@
 					(unit 1)
 				)
+			)
+		)
+	)
+	(symbol
+		(lib_id "Device:C_Small")
+		(at 44.45 49.53 180)
+		(unit 1)
+		(exclude_from_sim no)
+		(in_bom yes)
+		(on_board yes)
+		(dnp no)
+		(property "Reference" "C10"
+			(at 46.99 45.466 0)
+			(effects
+				(font
+					(size 1.27 1.27)
+				)
+			)
+		)
+		(property "Value" "100nF"
+			(at 48.768 47.498 0)
+			(effects
+				(font
+					(size 1.27 1.27)
+				)
+			)
+		)
+		(property "Footprint" "Capacitor_SMD:C_0805_2012Metric_Pad1.18x1.45mm_HandSolder"
+			(at 44.45 49.53 0)
+			(effects
+				(font
+					(size 1.27 1.27)
+				)
+				(hide yes)
+			)
+		)
+		(property "Datasheet" "~"
+			(at 44.45 49.53 0)
+			(effects
+				(font
+					(size 1.27 1.27)
+				)
+				(hide yes)
+			)
+		)
+		(property "Description" "Unpolarized capacitor, small symbol"
+			(at 44.45 49.53 0)
+			(effects
+				(font
+					(size 1.27 1.27)
+				)
+				(hide yes)
+			)
+		)
+		(pin "2"
+		)
+		(pin "1"
+		)
+		(instances
+			(project "KillSwitch"
+				(path "/722d8df3-08e9-470c-940d-01bb552f6a6b/dd4eb25e-e036-4865-9a65-d34df93aca5c"
+					(reference "C10")
+					(unit 1)
+				)
